File: CoarseSunSensor2.0/PhotodiodeArray.kicad_sch (KiCad schematic)
At the start: 13 parts

Commit message: Minor schematic changes
Calculei o valor dos capacitores e resistores
Parts:
- added C10: 10n, Capacitor_SMD:C_0603_1608Metric, symbol Device:C
- C1, C2, C3, C4: value C -> 150p
- R1, R2, R3, R4: value R -> 95k
Connections:
- net +3V3: now also C10.1
- net GND: now also C10.2
